File: RobotController.kicad_pcb (KiCad board)
At the start: 2 copper layers, 63 x 50.5 mm, 16 parts, among them J1 Rear Motor, J2 Left Motor, J3 Right Motor, U1 74HC14

Commit message: start version 0.2
Parts:
- removed ?: proto grid 14x4, Ferg Library:proto grid 14x4
- added J4: Head Encoder, Connector_JST:JST_PH_B3B-PH-K_1x03_P2.00mm_Vertical, B.Cu at (74.4, 33.0)
- J1: value Rear Motor -> Rear Encoder; footprint Connector_JST:JST_PH_S4B-PH-K_1x04_P2.00mm_Horizontal -> Connector_JST:JST_PH_B4B-PH-K_1x04_P2.00mm_Vertical
- J2: value Left Motor -> Left Encoder; footprint Connector_JST:JST_PH_S4B-PH-K_1x04_P2.00mm_Horizontal -> Connector_JST:JST_PH_B4B-PH-K_1x04_P2.00mm_Vertical
- J3: value Right Motor -> Right Encoder; footprint Connector_JST:JST_PH_S4B-PH-K_1x04_P2.00mm_Horizontal -> Connector_JST:JST_PH_B4B-PH-K_1x04_P2.00mm_Vertical
- R7, R8, R9: value 200 -> 100
- moved R3 31.0 mm to (28.2, 29.4), turned to 180 degrees
- moved R4 24.0 mm to (28.2, 32.6), turned to 180 degrees
- moved R7 21.8 mm to (68.6, 48.2)
- moved R2 21.7 mm to (45.4, 31.0), turned to 0 degrees
- moved R1 21.3 mm to (45.4, 27.6), turned to 0 degrees
- moved C1 21.2 mm to (45.4, 34.2), turned to 0 degrees
- moved U1 17.8 mm to (37.0, 30.0)
- moved R5 12.6 mm to (34.4, 37.0), turned to 180 degrees
- moved R6 12.6 mm to (39.8, 37.0)
- moved A1 3.99 mm to (63.6, 21.7)
- moved R8 3.58 mm to (27.8, 61.4)
- moved R9 3.41 mm to (27.8, 50.2)
- moved J1 1.22 mm to (74.4, 52.2)
- moved J3 1.06 mm to (22.2, 46.2)
- moved J2 1.05 mm to (22.2, 57.4)
Connections:
- A1 pad 16: unconnected-(A1-IO21-Pad16) -> Net-(A1-IO21)
Routing:
- net Net-(A1-IO21): track 0.00 -> 54.5 mm
- net +3V3: track 112.7 -> 144.7 mm, vias 0 -> 1
- net Net-(A1-IO4/A5): track 37.5 -> 11.8 mm
- net Net-(J1-Pin_3): track 26.6 -> 4.80 mm
- net Net-(J2-Pin_1): track 16.9 -> 38.5 mm, vias 0 -> 1
- net Net-(A1-IO36/A4): track 29.9 -> 11.8 mm
- net Net-(A1-I39/A3): track 29.6 -> 11.8 mm
- net Net-(A1-I34/A2): track 29.6 -> 11.8 mm
- net Net-(J2-Pin_2): track 30.6 -> 46.4 mm, vias 2 -> 1
- net Net-(J1-Pin_2): track 33.1 -> 43.8 mm
- net Net-(J3-Pin_1): track 20.9 -> 31.1 mm
- net Net-(J1-Pin_1): track 37.3 -> 46.9 mm
- net Net-(J3-Pin_2): track 17.4 -> 23.6 mm
- net Net-(A1-A7/IO32): track 14.9 -> 10.9 mm
- net Net-(A1-A6/IO14): track 13.8 -> 10.7 mm
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Other:
- board text added: "Forest Moon"
- board text added: "Rovio Motor Controller v0.2"

Commit message: kicad updates
Parts:
- J1: value Rear Encoder -> Rear
- J2: value Left Encoder -> Left
- J3: value Right Encoder -> Right
- J4: value Head Encoder -> Head
Changed lines of the file:
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@@
     (property "ki_keywords" "connector")
     (attr through_hole)
-    (fp_text reference "J2" (at 3 -2.9 -90) (layer "F.SilkS")
-        (effects (font (size 1 1) (thickness 0.15)))
-    )
-    (fp_text value "Left Encoder" (at 3 4 -90) (layer "F.Fab")
-        (effects (font (size 1 1) (thickness 0.15)))
-    )
-    (fp_text user "${REFERENCE}" (at 3 1.5 -90) (layer "F.Fab")
+    (fp_text reference "J2" (at 3 -2.9 90) (layer "F.SilkS")
+        (effects (font (size 1 1) (thickness 0.15)))
+    )
+    (fp_text value "Left" (at 3 4.2 90) (layer "F.SilkS")
+        (effects (font (size 1 1) (thickness 0.15)))
+    )
+    (fp_text user "${REFERENCE}" (at 3 1.5 90) (layer "F.Fab")
         (effects (font (size 1 1) (thickness 0.15)))
     )
@@
         (effects (font (size 1 1) (thickness 0.15)))
     )
-    (fp_text value "Rear Encoder" (at 3 4 90) (layer "F.Fab")
+    (fp_text value "Rear" (at 3 4.2 90) (layer "F.SilkS")
         (effects (font (size 1 1) (thickness 0.15)))
     )
@@
     (property "ki_keywords" "connector")
     (attr through_hole)
-    (fp_text reference "J3" (at 3 -2.9 -90) (layer "F.SilkS")
-        (effects (font (size 1 1) (thickness 0.15)))
-    )
-    (fp_text value "Right Encoder" (at 3 4 -90) (layer "F.Fab")
-        (effects (font (size 1 1) (thickness 0.15)))
-    )
-    (fp_text user "${REFERENCE}" (at 3 1.5 -90) (layer "F.Fab")
+    (fp_text reference "J3" (at 3 -2.9 90) (layer "F.SilkS")
+        (effects (font (size 1 1) (thickness 0.15)))
+    )
+    (fp_text value "Right" (at 3 4.4 90) (layer "F.SilkS")
+        (effects (font (size 1 1) (thickness 0.15)))
+    )
+    (fp_text user "${REFERENCE}" (at 3 1.5 90) (layer "F.Fab")
         (effects (font (size 1 1) (thickness 0.15)))
     )
@@
         (effects (font (size 1 1) (thickness 0.15)))
     )
-    (fp_text value "ESP32 Feather V2" (at 10.16 45.72 90) (layer "F.Fab")
+    (fp_text value "ESP32 Feather V2" (at 10.16 45.72 90) (layer "F.SilkS")
         (effects (font (size 1 1) (thickness 0.15)))
     )
@@
         (effects (font (size 1 1) (thickness 0.15)) (justify mirror))
     )
-    (fp_text value "Head Encoder" (at 2 -4 90) (layer "B.Fab")
+    (fp_text value "Head" (at 2 -4.2 90) (layer "B.SilkS")
         (effects (font (size 1 1) (thickness 0.15)) (justify mirror))
     )
